File: Schematic/Emat/Emat.brd (EAGLE design)
At the start: 100 x 80 mm, 42 parts, among them J1 PIN1-2, J2 PIN1-2, J3 PIN1-2, J4 PIN1-2, J5 PIN1-2, J8 PIN1-2, J9 PIN1-2, Q2 STP13NM60NTO247BV, U1 UCC27324D, X2 22-23-2021, X3 22-23-2021, X4 22-23-2021, X5 22-23-2021, X6 22-23-2021

Commit message: Fix schematic. 1.5KE300 added.
Parts:
- R9: value 510 -> 100
Changed lines of the file:
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@@
 <attribute name="MF" value="MOLEX" x="38.1" y="52.07" size="1.778" layer="28" rot="MR270" display="off"/>
 </element>
-<element name="R9" library="rcl" package="R1206" value="510" x="40.64" y="45.72"/>
+<element name="R9" library="rcl" package="R1206" value="100" x="40.64" y="45.72"/>
 <element name="X3" library="con-molex" package="22-23-2021" value="22-23-2021" x="49.53" y="43.18" rot="MR0">
 <attribute name="OC_NEWARK" value="25C3832" x="49.53" y="43.18" size="1.778" layer="28" rot="MR0" display="off"/>
